Commit message: back

File: ros/src/my_biped_robot_sims/urdf/biped.urdf (robot description, URDF)
Before this commit: robot biped, 9 links, 8 joints
Links:
- removed link L_contactsensor_link
- removed link R_contactsensor_link
- added link L_lowerleg_contactsensor_link, mass 0.0001; collision sphere radius=0.020; visual sphere radius=0.020
- added link R_lowerleg_contactsensor_link, mass 0.0001; collision sphere radius=0.020; visual sphere radius=0.020
- link L_hipassembly: geometry collision mesh filename=package://my_legged_robots_description/meshes/leg/hipassemb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 scale=1 1 1; visual mesh filename=package://my_legged_robots_description/meshes/leg/hipassemb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 scale=1 1 1
- link L_lowerleg: geometry collision mesh filename=package://my_legged_robots_description/meshes/leg/lowerleg.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 scale=1 1 1; visual mesh filename=package://my_legged_robots_description/meshes/leg/lowerleg.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 scale=1 1 1
- link L_upperleg: geometry collision mesh filename=package://my_legged_robots_description/meshes/leg/upperleg.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 scale=1 1 1; visual mesh filename=package://my_legged_robots_description/meshes/leg/upperleg.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 scale=1 1 1
- link R_hipassembly: geometry collision mesh filename=package://my_legged_robots_description/meshes/leg/hipassemb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 scale=1 1 1; visual mesh filename=package://my_legged_robots_description/meshes/leg/hipassemb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 scale=1 1 1
- link R_lowerleg: geometry collision mesh filename=package://my_legged_robots_description/meshes/leg/lowerleg.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 scale=1 1 1; visual mesh filename=package://my_legged_robots_description/meshes/leg/lowerleg.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 scale=1 1 1
- link R_upperleg: geometry collision mesh filename=package://my_legged_robots_description/meshes/leg/upperleg.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 scale=1 1 1; visual mesh filename=package://my_legged_robots_description/meshes/leg/upperleg.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 scale=1 1 1
- link base: geometry collision box size=0.20 0.20 0.30; visual box size=0.20 0.20 0.30
Joints:
- joint L_haa_joint: limit lower=-1.6 upper=1.6 effort=200 velocity=1.0 -> lower=-1.6 upper=1.6 effort=100 velocity=1.0; origin xyz=0.00000 0.1 -0.15000 rpy=2.0344439357957036 1.5707962290814481 -1.1071487177940917 -> xyz=0.0 0.1 -0.15000 rpy=2.0344439357957036 1.5707962290814481 -1.1071487177940917
- joint L_hfe_joint: limit lower=-1.6 upper=1.6 effort=200 velocity=1.0 -> lower=-1.6 upper=1.6 effort=100 velocity=1.0
- joint L_kfe_joint: limit lower=-1.6 upper=1.6 effort=200 velocity=1.0 -> lower=-1.6 upper=0.0 effort=100 velocity=1.0
- joint L_lowerleg_contactsensor_link_joint: child L_contactsensor_link -> L_lowerleg_contactsensor_link
- joint R_haa_joint: limit lower=-1.6 upper=1.6 effort=200 velocity=1.0 -> lower=-1.6 upper=1.6 effort=100 velocity=1.0; origin xyz=0.00000 -0.1 -0.15000 rpy=2.0344439357957036 1.5707962290814481 -1.1071487177940917 -> xyz=0.0 -0.1 -0.15000 rpy=2.0344439357957036 1.5707962290814481 -1.1071487177940917
- joint R_hfe_joint: limit lower=-1.6 upper=1.6 effort=200 velocity=1.0 -> lower=-1.6 upper=1.6 effort=100 velocity=1.0
- joint R_kfe_joint: limit lower=-1.6 upper=1.6 effort=200 velocity=1.0 -> lower=-1.6 upper=0.0 effort=100 velocity=1.0
- joint R_lowerleg_contactsensor_link_joint: child R_contactsensor_link -> R_lowerleg_contactsensor_link
